Commit message: Yaw-tuning round: R2 vs R3, promote Release_CandidateV2.1
Screened three reward levers for yaw wobble via 3M continuations from
Release_CandidateV2; the auto-picked winner (R2, paired FAC_YAW_TRACK +
FAC_RESID_SMOOTH) showed a live T5.2 regression on its own 3M sanity
check mid-schedule, so R3 (FAC_RESID_SMOOTH alone) was substituted and
both were finished to the same 13M-cumulative budget for a fair
comparison. R3 wins on every metric measured at equal budget, reversing
the 3M screening signal. Promoted to Release_CandidateV2.1.

Also folds in the getup-sim replay documentation and hardware-gated
backlog updates, and a batch of small pi_pipeline touch-ups (voice
effects layer, diag/feature-flag wiring) alongside the RL work.

File: rl_training/opencat-gym/models/bittle_esp32.urdf (robot description, URDF)
Before this commit: robot Bittle, 14 links, 13 joints
Joints:
- joint hip_left: limit lower=-1.57 upper=2.00 effort=0 velocity=0 -> lower=-1.57 upper=3.55 effort=0 velocity=0
- joint hip_right: limit lower=-1.57 upper=2.00 effort=0 velocity=0 -> lower=-1.57 upper=3.55 effort=0 velocity=0
- joint knee_left: limit lower=-1.57 upper=1.57 effort=0 velocity=0 -> lower=-1.57 upper=1.80 effort=0 velocity=0
- joint shoulder_left: limit lower=-1.57 upper=1.57 effort=0 velocity=0 -> lower=-3.15 upper=1.57 effort=0 velocity=0
- joint shoulder_right: limit lower=-1.57 upper=1.57 effort=0 velocity=0 -> lower=-3.15 upper=1.57 effort=0 velocity=0
